Commit message: use_des true, use_ekf delete
1. Delete use_ekf. robot rotate continuous if turn on ekf_node
2. use_des true by default
3. Reduce total.stl size to reduce loading time
4. Even don't use ekf_node, change ekf parameter not using IMU
5. Add robot on slamtoolbox rviz
6. delete remappings from cratographer lauch, not using ekf_node

File: monicar2_description/urdf/robot.urdf (robot description, URDF)
Before this commit: robot robot, 2 links, 1 joints
Links:
- link base_link: geometry visual mesh filename=package://monicar2_description/meshes/total.stl scale=0.001 0.001 0.001
